Commit message: Updated robot descriptions to match our physical differential drive robot to the nearest mm.

File: linorobot2_description/urdf/2wd_properties.urdf.xacro (robot description, xacro)
@@ -1,22 +1,26 @@
 <?xml version="1.0"?>
 <robot xmlns:xacro="http://ros.org/wiki/xacro">
-  <xacro:property name="base_length" value="0.24" />
-  <xacro:property name="base_width" value="0.275" />
-  <xacro:property name="base_height" value="0.003" />
-  <xacro:property name="base_mass" value="1" />
-  <xacro:property name="wheel_radius" value="0.045" />
-  <xacro:property name="wheel_width" value="0.01" />
-  <xacro:property name="wheel_pos_x" value="0.0" />
-  <xacro:property name="wheel_pos_y" value="0.13" />
-  <xacro:property name="wheel_pos_z" value="-0.03" />
-  <xacro:property name="wheel_mass" value=".1" />
-  <xacro:property name="wheel_torque" value="20" />
+  <xacro:property name="base_z_offset" value="0.011" />
+  <xacro:property name="base_col_height" value="0.057" />
+  <xacro:property name="base_bottom_height" value="0.031" />
+  <xacro:property name="base_pfm_thickness" value="0.003" />
+  <xacro:property name="base_inner_width" value="0.071" />
+  <xacro:property name="base_outer_width" value="0.126" />
+  <xacro:property name="base_length" value="0.150" />
+  <xacro:property name="base_width" value="${base_outer_width}" />
+  <xacro:property name="base_height" value=
+      "${base_bottom_height+base_bottom_height+base_pfm_thickness}" />
+  <xacro:property name="base_mass" value="0.5" />
+  <xacro:property name="wheel_radius" value="0.03" />
+  <xacro:property name="wheel_width" value="0.008" />
+  <xacro:property name="wheel_pos_x" value="0.005" />
+  <xacro:property name="wheel_pos_y" value="0.052" />
+  <xacro:property name="wheel_pos_z" value="-0.017" />
+  <xacro:property name="wheel_mass" value=".012" />
+  <xacro:property name="wheel_torque" value="1" />
   <xacro:property name="front_caster_wheel" value="true" />
-  <xacro:property name="rear_caster_wheel" value="true" />
+  <xacro:property name="rear_caster_wheel" value="false" />
   <xacro:property name="laser_pose">
-    <origin xyz="0.12 0 0.33" rpy="0 0 0"/>
-  </xacro:property>
-  <xacro:property name="depth_sensor_pose">
-    <origin xyz="0.14 0.0 0.045" rpy="0 0 0"/>
+    <origin xyz="0 0 ${base_height-base_z_offset}" rpy="0 0 0"/>
   </xacro:property>
 </robot>

File: linorobot2_description/urdf/mech/base.urdf.xacro (robot description, xacro)
@@ -1,11 +1,11 @@
 <?xml version="1.0"?>
 <robot xmlns:xacro="http://ros.org/wiki/xacro">
-  <xacro:macro name="base" params="length width height mass wheel_radius wheel_pos_z">
+  <xacro:macro name="base" params="length width height mass wheel_radius wheel_pos_z inner_width">
     <link name="base_footprint"/>
     <link name="base_link">
       <visual>
-        <origin xyz="0 0 0" rpy="0 0 0"/>
+        <origin xyz="0 0 ${base_z_offset}" rpy="0 0 0"/>
         <geometry>
-          <box size="${length} ${width} ${height}"/>
+          <box size="${length} ${inner_width} ${height}"/>
           <!-- <mesh filename="" scale="0.001 0.001 0.001"/> -->
         </geometry>
@@ -15,5 +15,5 @@
       </visual>
       <collision>
-        <origin xyz="0 0 0" rpy="0 0 0"/>
+        <origin xyz="0 0 ${base_z_offset}" rpy="0 0 0"/>
         <geometry>
           <box size="${length} ${width} ${height}"/>
@@ -21,7 +21,7 @@
       </collision>
       <inertial>
-        <origin xyz="0 0 0" rpy="0 0 0"/>
+        <origin xyz="0.02 0 0" rpy="0 0 0"/>
         <mass value="${mass}"/>
-        <inertia ixx="${(1/12) * mass * ((width  * width)  + (height * height))}" ixy="0.0" ixz="0.0"
+        <inertia ixx="${(1/12) * mass * ((width * width) + (height * height))}" ixy="0.0" ixz="0.0"
                  iyy="${(1/12) * mass * ((length * length) + (height * height))}" iyz="0.0"
                  izz="${(1/12) * mass * ((length * length) + (width  * width))}"/>

File: linorobot2_description/urdf/robots/2wd.urdf.xacro (robot description, xacro)
@@ -13,4 +13,5 @@
     width="${base_width}"
     height="${base_height}"
+    inner_width="${base_inner_width}"
     mass="${base_mass}"
     wheel_radius="${wheel_radius}"
@@ -57,7 +58,4 @@
     <xacro:insert_block name="laser_pose" />
   </xacro:generic_laser>
-  <xacro:depth_sensor>
-    <xacro:insert_block name="depth_sensor_pose" />
-  </xacro:depth_sensor>
   <xacro:diff_drive_controller
     wheel_separation="${wheel_pos_y * 2}"

File: linorobot2_description/urdf/sensors/imu.urdf.xacro (robot description, xacro)
@@ -5,5 +5,5 @@
       <parent link="base_link"/>
       <child link="imu_link"/>
-      <origin xyz="0 0 0" rpy="0 0 0"/>
+      <origin xyz="0.01 0 0" rpy="0 0 0"/>
     </joint>
     <gazebo reference="imu_link">

File: linorobot2_description/urdf/sensors/laser.urdf.xacro (robot description, xacro)
@@ -4,7 +4,7 @@
     <link name="${frame_id}">
       <visual>
-        <origin xyz="0 0 -0.025" rpy="0 0 0"/>
+        <origin xyz="0 0 0" rpy="0 0 0"/>
         <geometry>
-          <cylinder radius="0.0375" length="0.05"/>
+          <cylinder radius="0.032" length="0.016"/>
         </geometry>
         <material name="green">
@@ -13,7 +13,7 @@
       </visual>
       <collision>
-        <origin xyz="0 0 -0.025" rpy="0 0 0"/>
+        <origin xyz="0 0 0" rpy="0 0 0"/>
         <geometry>
-          <cylinder radius="0.0375" length="0.05"/>
+          <cylinder radius="0.04" length="0.016"/>
         </geometry>
       </collision>

Commit message: Updated robot description and created accurate mesh of physical robot.

File: linorobot2_description/urdf/2wd_properties.urdf.xacro (robot description, xacro)
@@ -4,12 +4,14 @@
   <xacro:property name="base_col_height" value="0.057" />
   <xacro:property name="base_bottom_height" value="0.031" />
-  <xacro:property name="base_pfm_thickness" value="0.003" />
+  <xacro:property name="base_pfm_height" value="0.003" />
   <xacro:property name="base_inner_width" value="0.071" />
   <xacro:property name="base_outer_width" value="0.126" />
-  <xacro:property name="base_length" value="0.150" />
+  <xacro:property name=
+  "base_length" value="0.150" />
   <xacro:property name="base_width" value="${base_outer_width}" />
   <xacro:property name="base_height" value=
-      "${base_bottom_height+base_bottom_height+base_pfm_thickness}" />
-  <xacro:property name="base_mass" value="0.5" />
+      "${base_bottom_height+base_col_height+base_pfm_height
+  }" />
+  <xacro:property name="base_mass" value="2" />
   <xacro:property name="wheel_radius" value="0.03" />
   <xacro:property name="wheel_width" value="0.008" />
@@ -17,10 +19,10 @@
   <xacro:property name="wheel_pos_y" value="0.052" />
   <xacro:property name="wheel_pos_z" value="-0.017" />
-  <xacro:property name="wheel_mass" value=".012" />
+  <xacro:property name="wheel_mass" value="0.01" />
   <xacro:property name="wheel_torque" value="1" />
   <xacro:property name="front_caster_wheel" value="true" />
   <xacro:property name="rear_caster_wheel" value="false" />
   <xacro:property name="laser_pose">
-    <origin xyz="0 0 ${base_height-base_z_offset}" rpy="0 0 0"/>
+    <origin xyz="0 0 ${base_col_height}" rpy="0 0 0"/>
   </xacro:property>
 </robot>

File: linorobot2_description/urdf/controllers/diff_drive.urdf.xacro (robot description, xacro)
@@ -11,4 +11,5 @@
         <wheel_separation>${wheel_separation}</wheel_separation>
         <wheel_diameter>${wheel_radius * 2}</wheel_diameter>
+        <wheel_torque>${wheel_torque}</wheel_torque>
         <max_wheel_acceleration>1.0</max_wheel_acceleration>
         <robot_base_frame>base_footprint</robot_base_frame>

File: linorobot2_description/urdf/mech/base.urdf.xacro (robot description, xacro)
@@ -5,11 +5,11 @@
     <link name="base_link">
       <visual>
-        <origin xyz="0 0 ${base_z_offset}" rpy="0 0 0"/>
+        <origin xyz="0 0 -0.006" rpy="0 0 0"/>
         <geometry>
-          <box size="${length} ${inner_width} ${height}"/>
-          <!-- <mesh filename="" scale="0.001 0.001 0.001"/> -->
+          <!-- <box size="${length} ${inner_width} ${height}"/> -->
+          <mesh filename="package://linorobot2_description/urdf/meshes/capstone_mesh_FRU.stl" scale="0.001 0.001 0.001"/>
         </geometry>
-        <material name="yellow">
-          <color rgba="0.8784 0.6627 0.6627 1.0"/>
+        <material name="gray">
+          <color rgba="0.5 0.5 0.5 1.0"/>
         </material>
       </visual>
@@ -21,9 +21,9 @@
       </collision>
       <inertial>
-        <origin xyz="0.02 0 0" rpy="0 0 0"/>
+        <origin xyz="0.022 0 0" rpy="0 0 0"/>
         <mass value="${mass}"/>
-        <inertia ixx="${(1/12) * mass * ((width * width) + (height * height))}" ixy="0.0" ixz="0.0"
-                 iyy="${(1/12) * mass * ((length * length) + (height * height))}" iyz="0.0"
-                 izz="${(1/12) * mass * ((length * length) + (width  * width))}"/>
+        <inertia ixx="${(4/12) * mass * ((width * width) + (height * height))}" ixy="0.0" ixz="0.0"
+                 iyy="${(4/12) * mass * ((length * length) + (height * height))}" iyz="0.0"
+                 izz="${(4/12) * mass * ((length * length) + (width  * width))}"/>
       </inertial>
     </link>

File: linorobot2_description/urdf/mech/wheel.urdf.xacro (robot description, xacro)
@@ -8,6 +8,6 @@
           <cylinder radius="${radius}" length="${width}"/>
         </geometry>
-        <material name="blue">
-            <color rgba="0.1764 0.4588 0.8509 1.0"/>
+        <material name="black">
+            <color rgba="0.0 0.0 0.0 1.0"/>
         </material>
       </visual>
@@ -29,10 +29,14 @@
       <visual>
         <material>
-          <ambient>0.1764 0.4588 0.8509 1.0</ambient>
-          <diffuse>0.1764 0.4588 0.8509 1.0</diffuse>
-          <specular>0.1764 0.4588 0.8509 1.0</specular>
+          <ambient>0.0 0.0 0.0 1.0</ambient>
+          <diffuse>0.0 0.0 0.0 1.0</diffuse>
+          <specular>0.0 0.0 0.0 1.0</specular>
           <emissive>0.0 0.0 0.0 0.0</emissive>
         </material>
       </visual>
+      <!-- <mu1>0.9</mu1>
+      <mu2>0.9</mu2>   -->
+      <!-- <kp>1000</kp>
+      <kd>1</kd> -->
     </gazebo>
     <joint name="${side}_wheel_joint" type="continuous">

File: linorobot2_description/urdf/sensors/generic_laser.urdf.xacro (robot description, xacro)
@@ -8,6 +8,6 @@
       min_angle="-3.1416"
       max_angle="3.1416"
-      min_range="0.08"
-      max_range="12.0"
+      min_range="0.12"
+      max_range="3.5"
       frame_id="laser"
       topic_name="scan"

File: linorobot2_description/urdf/sensors/laser.urdf.xacro (robot description, xacro)
@@ -4,16 +4,16 @@
     <link name="${frame_id}">
       <visual>
-        <origin xyz="0 0 0" rpy="0 0 0"/>
+        <origin xyz="0 0 0.019" rpy="0 0 0"/>
         <geometry>
-          <cylinder radius="0.032" length="0.016"/>
+          <cylinder radius="0.033" length="0.038"/>
         </geometry>
-        <material name="green">
-            <color rgba="0.003 0.639 0.223 1.0"/>
+        <material name="black">
+            <color rgba="0.0 0.0 0.0 1.0"/>
         </material>
       </visual>
       <collision>
-        <origin xyz="0 0 0" rpy="0 0 0"/>
+        <origin xyz="0 0 0.019" rpy="0 0 0"/>
         <geometry>
-          <cylinder radius="0.04" length="0.016"/>
+          <box size=".095 0.066 0.04" length="0.016"/>
         </geometry>
       </collision>
@@ -29,7 +29,7 @@
       <visual>
         <material>
-          <ambient>0.003 0.639 0.223 1.0</ambient>
-          <diffuse>0.003 0.639 0.223 1.0</diffuse>
-          <specular>0.003 0.639 0.223 1.0</specular>
+          <ambient>0.0 0.0 0.0 1.0</ambient>
+          <diffuse>0.0 0.0 0.0 1.0</diffuse>
+          <specular>0.0 0.0 0.0 1.0</specular>
           <emissive>0.0 0.0 0.0 0.0</emissive>
         </material>

Commit message: Removed unnecessary description files. Updated Xacro.

File: linorobot2_description/urdf/2wd_properties.urdf.xacro (robot description, xacro)
@@ -1,7 +1,7 @@
 <?xml version="1.0"?>
 <robot xmlns:xacro="http://ros.org/wiki/xacro">
-  <xacro:property name="base_z_offset" value="0.011" />
+  <xacro:property name="base_z_offset" value="0.016" />
   <xacro:property name="base_col_height" value="0.057" />
-  <xacro:property name="base_bottom_height" value="0.031" />
+  <xacro:property name="base_bottom_height" value="0.032" />
   <xacro:property name="base_pfm_height" value="0.003" />
   <xacro:property name="base_inner_width" value="0.071" />

File: linorobot2_description/urdf/controllers/diff_drive.urdf.xacro (robot description, xacro)
@@ -13,9 +13,11 @@
         <wheel_torque>${wheel_torque}</wheel_torque>
         <max_wheel_acceleration>1.0</max_wheel_acceleration>
-        <robot_base_frame>base_footprint</robot_base_frame>
+        <robot_base_frame>base_link</robot_base_frame>
         <publish_odom>true</publish_odom>
         <publish_odom_tf>false</publish_odom_tf>
         <publish_wheel_tf>true</publish_wheel_tf>
         <odometry_frame>odom</odometry_frame>
+        <mu1>0.9</mu1>
+        <mu2>0.9</mu2>
       </plugin>
     </gazebo>

File: linorobot2_description/urdf/controllers/skid_steer.urdf.xacro (robot description, xacro)
@@ -17,5 +17,5 @@
         <updateRate>100</updateRate>
         <max_wheel_acceleration>1.0</max_wheel_acceleration>
-        <robot_base_frame>base_footprint</robot_base_frame>
+        <robot_base_frame>base_link</robot_base_frame>
         <publish_odom>true</publish_odom>
         <publish_odom_tf>false</publish_odom_tf>

File: linorobot2_description/urdf/mech/base.urdf.xacro (robot description, xacro)
@@ -8,5 +8,5 @@
         <geometry>
           <!-- <box size="${length} ${inner_width} ${height}"/> -->
-          <mesh filename="package://linorobot2_description/urdf/meshes/capstone_mesh_FRU.stl" scale="0.001 0.001 0.001"/>
+          <mesh filename="file://$(find linorobot2_description)/urdf/meshes/capstone_mesh_FRU.stl" scale="0.001 0.001 0.001"/>
         </geometry>
         <material name="gray">

File: linorobot2_description/urdf/mech/caster_wheel.urdf.xacro (robot description, xacro)
@@ -34,4 +34,10 @@
     </link>
     <gazebo reference="${side}_caster_wheel_link">
+        <material>
+          <ambient>0.1 0.1 0.1 1.0</ambient>
+          <diffuse>0.1 0.1 0.1 1.0</diffuse>
+          <specular>0.1 0.1 0.1 1.0</specular>
+          <emissive>0.1 0.1 0.1 1.0</emissive>
+        </material>
         <mu1>0.01</mu1>
         <mu2>0.01</mu2>

File: linorobot2_description/urdf/mech/wheel.urdf.xacro (robot description, xacro)
@@ -27,16 +27,14 @@
     </link>
     <gazebo reference="${side}_wheel_link">
+      <mu1>0.2</mu1>
+      <mu2>0.2</mu2>
       <visual>
         <material>
-          <ambient>0.0 0.0 0.0 1.0</ambient>
-          <diffuse>0.0 0.0 0.0 1.0</diffuse>
-          <specular>0.0 0.0 0.0 1.0</specular>
-          <emissive>0.0 0.0 0.0 0.0</emissive>
+          <ambient>0.1 0.1 0.1 1.0</ambient>
+          <diffuse>0.1 0.1 0.1 1.0</diffuse>
+          <specular>0.1 0.1 0.1 1.0</specular>
+          <emissive>0.1 0.1 0.1 1.0</emissive>
         </material>
       </visual>
-      <!-- <mu1>0.9</mu1>
-      <mu2>0.9</mu2>   -->
-      <!-- <kp>1000</kp>
-      <kd>1</kd> -->
     </gazebo>
     <joint name="${side}_wheel_joint" type="continuous">

File: linorobot2_description/urdf/sensors/imu.urdf.xacro (robot description, xacro)
@@ -15,15 +15,15 @@
       <topic>__default_topic__</topic>
       <plugin filename="libgazebo_ros_imu_sensor.so" name="imu_plugin">
-          <ros>
-            <remapping>~/out:=imu/data</remapping>
-          </ros>
-          <topicName>imu/data</topicName>
-          <bodyName>imu_link</bodyName>
-          <updateRateHZ>10.0</updateRateHZ>
-          <gaussianNoise>0.0</gaussianNoise>
-          <xyzOffset>0 0 0</xyzOffset>
-          <rpyOffset>0 0 0</rpyOffset>
-          <frameName>imu_link</frameName>
-          <initialOrientationAsReference>false</initialOrientationAsReference>
+        <ros>
+          <remapping>~/out:=imu/data</remapping>
+        </ros>
+        <initialOrientationAsReference>false</initialOrientationAsReference>
+        <topicName>imu/data</topicName>
+        <bodyName>imu_link</bodyName>
+        <updateRateHZ>10.0</updateRateHZ>
+        <gaussianNoise>0.0</gaussianNoise>
+        <xyzOffset>0 0 0</xyzOffset>
+        <rpyOffset>0 0 0</rpyOffset>
+        <frameName>imu_link</frameName>
       </plugin>
       <pose>0 0 0 0 0 0</pose>
