Commit message: Updated configuration. SLAM functionality working as expected.

File: linorobot2_description/urdf/controllers/diff_drive.urdf.xacro (robot description, xacro)
@@ -6,4 +6,5 @@
           <argument>odom:=odom/unfiltered</argument>
         </ros>
+        <robot_base_frame>base_link</robot_base_frame>
         <updateRate>100</updateRate>
         <left_joint>left_wheel_joint</left_joint>
@@ -13,11 +14,10 @@
         <wheel_torque>${wheel_torque}</wheel_torque>
         <max_wheel_acceleration>1.0</max_wheel_acceleration>
-        <robot_base_frame>base_link</robot_base_frame>
         <publish_odom>true</publish_odom>
         <publish_odom_tf>false</publish_odom_tf>
         <publish_wheel_tf>true</publish_wheel_tf>
         <odometry_frame>odom</odometry_frame>
-        <mu1>0.9</mu1>
-        <mu2>0.9</mu2>
+        <mu1>0.5</mu1>
+        <mu2>0.5</mu2>
       </plugin>
     </gazebo>

File: linorobot2_description/urdf/controllers/skid_steer.urdf.xacro (robot description, xacro)
@@ -22,4 +22,8 @@
         <publish_wheel_tf>true</publish_wheel_tf>
         <odometry_frame>odom</odometry_frame>
+        <mu1>0.5</mu1>
+        <mu2>0.5</mu2>
+        <kp>10</kp>
+        <kd>1</kd>
       </plugin>
     </gazebo>

File: linorobot2_description/urdf/mech/base.urdf.xacro (robot description, xacro)
@@ -10,6 +10,6 @@
           <mesh filename="file://$(find linorobot2_description)/urdf/meshes/capstone_mesh_FRU.stl" scale="0.001 0.001 0.001"/>
         </geometry>
-        <material name="gray">
-          <color rgba="0.5 0.5 0.5 1.0"/>
+        <material name="white">
+          <color rgba="1 1 1 1.0"/>
         </material>
       </visual>
@@ -31,8 +31,8 @@
       <visual>
         <material>
-          <ambient>0.8392 0.6314 0.0 1.0</ambient>
-          <diffuse>0.8392 0.6314 0.0 1.0</diffuse>
+          <ambient>1 1 1 1.0</ambient>
+          <diffuse>1 1 1 1.0</diffuse>
           <specular>0.99 0.99 0.99 1.0</specular>
-          <emissive>0.0 0.0 0.0 0.0</emissive>
+          <emissive>0.5 0.5 0.5 0.0</emissive>
         </material>
       </visual>

File: linorobot2_description/urdf/mech/caster_wheel.urdf.xacro (robot description, xacro)
@@ -15,6 +15,6 @@
           <sphere radius="${caster_wheel_radius}" />
         </geometry>
-        <material name="black">
-            <color rgba="0.0 0.0 0.0 1.0"/>
+        <material name="gray">
+            <color rgba="0.1 0.1 0.1 1.0"/>
         </material>
       </visual>
@@ -34,4 +34,5 @@
     </link>
     <gazebo reference="${side}_caster_wheel_link">
+      <visual/>
         <material>
           <ambient>0.1 0.1 0.1 1.0</ambient>
@@ -40,6 +41,7 @@
           <emissive>0.1 0.1 0.1 1.0</emissive>
         </material>
-        <mu1>0.01</mu1>
-        <mu2>0.01</mu2>
+      <visual/>
+      <mu1>0.01</mu1>
+      <mu2>0.01</mu2>
     </gazebo>
     <joint name="${side}_caster_wheel_joint" type="fixed">

File: linorobot2_description/urdf/mech/wheel.urdf.xacro (robot description, xacro)
@@ -8,6 +8,6 @@
           <cylinder radius="${radius}" length="${width}"/>
         </geometry>
-        <material name="black">
-            <color rgba="0.0 0.0 0.0 1.0"/>
+        <material name="gray">
+            <color rgba="0.1 0.1 0.1 1.0"/>
         </material>
       </visual>
@@ -27,6 +27,4 @@
     </link>
     <gazebo reference="${side}_wheel_link">
-      <mu1>0.2</mu1>
-      <mu2>0.2</mu2>
       <visual>
         <material>

File: linorobot2_description/urdf/robots/2wd.urdf.xacro (robot description, xacro)
@@ -7,5 +7,4 @@
   <xacro:include filename="$(find linorobot2_description)/urdf/sensors/imu.urdf.xacro" />
   <xacro:include filename="$(find linorobot2_description)/urdf/sensors/generic_laser.urdf.xacro" />
-  <xacro:include filename="$(find linorobot2_description)/urdf/sensors/depth_sensor.urdf.xacro" />
   <xacro:include filename="$(find linorobot2_description)/urdf/controllers/diff_drive.urdf.xacro" />
   <xacro:base
@@ -45,13 +44,4 @@
     />
   </xacro:if>
-  <xacro:if value="${rear_caster_wheel}">
-    <xacro:caster_wheel
-      side="rear"
-      mass="0.01"
-      base_length="${base_length}"
-      wheel_radius="${wheel_radius}"
-      wheel_pos_z="${wheel_pos_z}"
-    />
-  </xacro:if>
   <xacro:imu/>
   <xacro:generic_laser>

File: linorobot2_description/urdf/sensors/imu.urdf.xacro (robot description, xacro)
@@ -5,5 +5,5 @@
       <parent link="base_link"/>
       <child link="imu_link"/>
-      <origin xyz="0.01 0 0" rpy="0 0 0"/>
+      <origin xyz="0 0 0" rpy="0 0 0"/>
     </joint>
     <gazebo reference="imu_link">
@@ -26,4 +26,9 @@
         <rpyOffset>0 0 0</rpyOffset>
         <frameName>imu_link</frameName>
+        <noise>
+          <type>gaussian</type>
+          <mean>0.0</mean>
+          <stddev>0.001</stddev>
+        </noise>
       </plugin>
       <pose>0 0 0 0 0 0</pose>

Commit message: Implemented separate namespaces to separate robot transform frames.

File: linorobot2_description/urdf/controllers/diff_drive.urdf.xacro (robot description, xacro)
@@ -1,4 +1,4 @@
 <robot xmlns:xacro="http://ros.org/wiki/xacro">
-  <xacro:macro name="diff_drive_controller" params="wheel_separation wheel_radius wheel_torque">
+  <xacro:macro name="diff_drive_controller" params="prefix wheel_separation wheel_radius wheel_torque">
     <gazebo>
       <plugin name="differential_drive_controller" filename="libgazebo_ros_diff_drive.so">
@@ -6,8 +6,8 @@
           <argument>odom:=odom/unfiltered</argument>
         </ros>
-        <robot_base_frame>base_link</robot_base_frame>
+        <robot_base_frame>base_link${prefix}</robot_base_frame>
         <updateRate>100</updateRate>
-        <left_joint>left_wheel_joint</left_joint>
-        <right_joint>right_wheel_joint</right_joint>
+        <left_joint>left_wheel_joint${prefix}</left_joint>
+        <right_joint>right_wheel_joint${prefix}</right_joint>
         <wheel_separation>${wheel_separation}</wheel_separation>
         <wheel_diameter>${wheel_radius * 2}</wheel_diameter>
@@ -17,5 +17,5 @@
         <publish_odom_tf>false</publish_odom_tf>
         <publish_wheel_tf>true</publish_wheel_tf>
-        <odometry_frame>odom</odometry_frame>
+        <odometry_frame>odom${prefix}</odometry_frame>
         <mu1>0.5</mu1>
         <mu2>0.5</mu2>

File: linorobot2_description/urdf/mech/base.urdf.xacro (robot description, xacro)
@@ -1,7 +1,7 @@
 <?xml version="1.0"?>
 <robot xmlns:xacro="http://ros.org/wiki/xacro">
-  <xacro:macro name="base" params="length width height mass wheel_radius wheel_pos_z inner_width">
-    <link name="base_footprint"/>
-    <link name="base_link">
+  <xacro:macro name="base" params="prefix length width height mass wheel_radius wheel_pos_z inner_width">
+    <link name="base_footprint${prefix}"/>
+    <link name="base_link${prefix}">
       <visual>
         <origin xyz="0 0 -0.006" rpy="0 0 0"/>
@@ -28,5 +28,5 @@
       </inertial>
     </link>
-    <gazebo reference="base_link">
+    <gazebo reference="base_link${prefix}">
       <visual>
         <material>
@@ -38,7 +38,7 @@
       </visual>
     </gazebo>
-    <joint name="base_to_footprint" type="fixed">
-      <parent link="base_footprint"/>
-      <child link="base_link"/>
+    <joint name="base_to_footprint${prefix}" type="fixed">
+      <parent link="base_footprint${prefix}"/>
+      <child link="base_link${prefix}"/>
       <origin xyz="0 0 ${wheel_radius - wheel_pos_z}" rpy="0 0 0"/>
     </joint>

File: linorobot2_description/urdf/mech/caster_wheel.urdf.xacro (robot description, xacro)
@@ -1,5 +1,5 @@
 <?xml version="1.0"?>
 <robot xmlns:xacro="http://ros.org/wiki/xacro">
-  <xacro:macro name="caster_wheel" params="side mass base_length wheel_radius wheel_pos_z">
+  <xacro:macro name="caster_wheel" params="prefix side mass base_length wheel_radius wheel_pos_z">
     <xacro:property name="caster_wheel_radius" value="${(wheel_radius - wheel_pos_z) / 2}" />
     <xacro:if value="${side == 'front'}">
@@ -9,5 +9,5 @@
         <xacro:property name="caster_wheel_x" value="${-(base_length / 2) + caster_wheel_radius}" />
     </xacro:if>
-    <link name="${side}_caster_wheel_link">
+    <link name="${side}_caster_wheel_link${prefix}">
       <visual>
         <origin xyz="0 0 0" rpy="0 0 0"/>
@@ -33,5 +33,5 @@
       </inertial>
     </link>
-    <gazebo reference="${side}_caster_wheel_link">
+    <gazebo reference="${side}_caster_wheel_link${prefix}">
       <visual/>
         <material>
@@ -45,7 +45,7 @@
       <mu2>0.01</mu2>
     </gazebo>
-    <joint name="${side}_caster_wheel_joint" type="fixed">
-      <parent link="base_link"/>
-      <child link="${side}_caster_wheel_link"/>
+    <joint name="${side}_caster_wheel_joint${prefix}" type="fixed">
+      <parent link="base_link${prefix}"/>
+      <child link="${side}_caster_wheel_link${prefix}"/>
       <origin xyz="${caster_wheel_x} 0 -${caster_wheel_radius}" rpy="0 0 0"/>
     </joint>

File: linorobot2_description/urdf/mech/wheel.urdf.xacro (robot description, xacro)
@@ -1,6 +1,6 @@
 <?xml version="1.0"?>
 <robot xmlns:xacro="http://ros.org/wiki/xacro">
-  <xacro:macro name="wheel" params="side radius width pos_x pos_y pos_z mass">
-    <link name="${side}_wheel_link">
+  <xacro:macro name="wheel" params="prefix side radius width pos_x pos_y pos_z mass">
+    <link name="${side}_wheel_link${prefix}">
       <visual>
         <origin xyz="0 0 0" rpy="${pi/2} 0 0"/>
@@ -26,5 +26,5 @@
       </inertial>
     </link>
-    <gazebo reference="${side}_wheel_link">
+    <gazebo reference="${side}_wheel_link${prefix}">
       <visual>
         <material>
@@ -36,8 +36,8 @@
       </visual>
     </gazebo>
-    <joint name="${side}_wheel_joint" type="continuous">
+    <joint name="${side}_wheel_joint${prefix}" type="continuous">
       <axis xyz="0 1 0" />
-      <parent link="base_link"/>
-      <child link="${side}_wheel_link"/>
+      <parent link="base_link${prefix}"/>
+      <child link="${side}_wheel_link${prefix}"/>
       <origin xyz="${pos_x} ${pos_y} ${pos_z}" rpy="0 0 0"/>
     </joint>

File: linorobot2_description/urdf/robots/2wd.urdf.xacro (robot description, xacro)
@@ -1,4 +1,4 @@
 <?xml version="1.0"?>
-<robot name="linorobot2_2wd" xmlns:xacro="http://ros.org/wiki/xacro">
+<robot xmlns:xacro="http://ros.org/wiki/xacro">
   <xacro:include filename="$(find linorobot2_description)/urdf/2wd_properties.urdf.xacro" />
   <xacro:include filename="$(find linorobot2_description)/urdf/mech/base.urdf.xacro" />
@@ -8,48 +8,57 @@
   <xacro:include filename="$(find linorobot2_description)/urdf/sensors/generic_laser.urdf.xacro" />
   <xacro:include filename="$(find linorobot2_description)/urdf/controllers/diff_drive.urdf.xacro" />
-  <xacro:base
-    length="${base_length}"
-    width="${base_width}"
-    height="${base_height}"
-    inner_width="${base_inner_width}"
-    mass="${base_mass}"
-    wheel_radius="${wheel_radius}"
-    wheel_pos_z="${wheel_pos_z}"
-/>
-  <xacro:wheel
-    side="left"
-    radius="${wheel_radius}"
-    width="${wheel_width}"
-    pos_x="${wheel_pos_x}"
-    pos_y="${wheel_pos_y}"
-    pos_z="${wheel_pos_z}"
-    mass="${wheel_mass}"
-  />
-  <xacro:wheel
-    side="right"
-    radius="${wheel_radius}"
-    width="${wheel_width}"
-    pos_x="${wheel_pos_x}"
-    pos_y="${-wheel_pos_y}"
-    pos_z="${wheel_pos_z}"
-    mass="${wheel_mass}"
-  />
-  <xacro:if value="${front_caster_wheel}">
-    <xacro:caster_wheel
-      side="front"
-      mass="0.01"
-      base_length="${base_length}"
+  <xacro:macro name="linorobot2_2wd" params="prefix">
+    <xacro:base
+      prefix="${prefix}"
+      length="${base_length}"
+      width="${base_width}"
+      height="${base_height}"
+      inner_width="${base_inner_width}"
+      mass="${base_mass}"
       wheel_radius="${wheel_radius}"
       wheel_pos_z="${wheel_pos_z}"
     />
-  </xacro:if>
-  <xacro:imu/>
-  <xacro:generic_laser>
-    <xacro:insert_block name="laser_pose" />
-  </xacro:generic_laser>
-  <xacro:diff_drive_controller
-    wheel_separation="${wheel_pos_y * 2}"
-    wheel_radius="${wheel_radius}"
-    wheel_torque="${wheel_torque}"
-  />
+    <xacro:wheel
+      prefix="${prefix}"
+      side="left"
+      radius="${wheel_radius}"
+      width="${wheel_width}"
+      pos_x="${wheel_pos_x}"
+      pos_y="${wheel_pos_y}"
+      pos_z="${wheel_pos_z}"
+      mass="${wheel_mass}"
+    />
+    <xacro:wheel
+      prefix="${prefix}"
+      side="right"
+      radius="${wheel_radius}"
+      width="${wheel_width}"
+      pos_x="${wheel_pos_x}"
+      pos_y="${-wheel_pos_y}"
+      pos_z="${wheel_pos_z}"
+      mass="${wheel_mass}"
+    />
+    <xacro:if value="${front_caster_wheel}">
+      <xacro:caster_wheel
+        prefix="${prefix}"
+        side="front"
+        mass="0.01"
+        base_length="${base_length}"
+        wheel_radius="${wheel_radius}"
+        wheel_pos_z="${wheel_pos_z}"
+      />
+    </xacro:if>
+    <xacro:imu
+      prefix="${prefix}"
+    />
+    <xacro:generic_laser prefix="${prefix}">
+      <xacro:insert_block name="laser_pose"/>
+    </xacro:generic_laser>
+    <xacro:diff_drive_controller
+      prefix="${prefix}"
+      wheel_separation="${wheel_pos_y * 2}"
+      wheel_radius="${wheel_radius}"
+      wheel_torque="${wheel_torque}"
+    />
+  </xacro:macro>
 </robot>

File: linorobot2_description/urdf/sensors/generic_laser.urdf.xacro (robot description, xacro)
@@ -2,7 +2,8 @@
 <robot xmlns:xacro="http://ros.org/wiki/xacro">
   <xacro:include filename="$(find linorobot2_description)/urdf/sensors/laser.urdf.xacro" />
-  <xacro:macro name="generic_laser" params="*origin">
+  <xacro:macro name="generic_laser" params="prefix *origin">
     <xacro:laser
-      update_rate="10"
+      prefix="${prefix}"
+      update_rate="1"
       ray_count="360"
       min_angle="-3.1416"
@@ -16,7 +17,8 @@
     </xacro:laser>
   </xacro:macro>
-  <xacro:macro name="generic_base_laser" params="*origin">
+  <xacro:macro name="generic_base_laser" params="prefix *origin">
     <xacro:laser
-      update_rate="10"
+      prefix="${prefix}"
+      update_rate="1"
       ray_count="360"
       min_angle="-3.1416"

File: linorobot2_description/urdf/sensors/imu.urdf.xacro (robot description, xacro)
@@ -1,11 +1,11 @@
 <robot xmlns:xacro="http://ros.org/wiki/xacro">
-  <xacro:macro name="imu">
-    <link name="imu_link"/>
-    <joint name="imu_to_base_link" type="fixed">
-      <parent link="base_link"/>
-      <child link="imu_link"/>
+  <xacro:macro name="imu" params="prefix">
+    <link name="imu_link${prefix}"/>
+    <joint name="imu_to_base_link${prefix}" type="fixed">
+      <parent link="base_link${prefix}"/>
+      <child link="imu_link${prefix}"/>
       <origin xyz="0 0 0" rpy="0 0 0"/>
     </joint>
-    <gazebo reference="imu_link">
+    <gazebo reference="imu_link${prefix}">
       <gravity>true</gravity>
       <sensor name="imu_sensor" type="imu">

File: linorobot2_description/urdf/sensors/laser.urdf.xacro (robot description, xacro)
@@ -1,6 +1,6 @@
 <robot xmlns:xacro="http://ros.org/wiki/xacro">
   <xacro:property name="M_PI" value="3.1415926535897931" />
-  <xacro:macro name="laser" params="*origin update_rate ray_count min_angle max_angle min_range max_range frame_id topic_name">
-    <link name="${frame_id}">
+  <xacro:macro name="laser" params="prefix *origin update_rate ray_count min_angle max_angle min_range max_range frame_id topic_name">
+    <link name="${frame_id}${prefix}">
       <visual>
         <origin xyz="0 0 0.019" rpy="0 0 0"/>
@@ -26,5 +26,5 @@
       </inertial>
     </link>
-    <gazebo reference="${frame_id}">
+    <gazebo reference="${frame_id}${prefix}">
       <visual>
         <material>
@@ -36,10 +36,10 @@
       </visual>
     </gazebo>
-    <joint name="${frame_id}_to_base_link" type="fixed">
-      <parent link="base_link"/>
-      <child link="${frame_id}"/>
+    <joint name="${frame_id}_to_base_link${prefix}" type="fixed">
+      <parent link="base_link${prefix}"/>
+      <child link="${frame_id}${prefix}"/>
       <xacro:insert_block name="origin" />
     </joint>
-    <gazebo reference="${frame_id}">
+    <gazebo reference="${frame_id}${prefix}">
       <sensor type="ray" name="${frame_id}_head_hokuyo_sensor">
         <always_on>true</always_on>
