Commit message: Robot spawns and pubs odom from ekf node in simulation for both namespaced and non-namespaced agents.

File: fru_bot_description/urdf/2wd_properties.urdf.xacro (robot description, xacro)
@@ -13,5 +13,5 @@
       "${base_bottom_height+base_col_height+base_pfm_height
   }" />
-  <xacro:property name="base_mass" value="2" />
+  <xacro:property name="base_mass" value="0.54" />
   <xacro:property name="wheel_radius" value="0.03" />
   <xacro:property name="wheel_width" value="0.008" />
@@ -20,5 +20,5 @@
   <xacro:property name="wheel_pos_z" value="-0.017" />
   <xacro:property name="wheel_mass" value="0.01" />
-  <xacro:property name="wheel_torque" value="1" />
+  <xacro:property name="wheel_torque" value="0.84" />
   <xacro:property name="front_caster_wheel" value="true" />
   <xacro:property name="rear_caster_wheel" value="false" />

File: fru_bot_description/urdf/controllers/diff_drive.urdf.xacro (robot description, xacro)
@@ -8,5 +8,5 @@
         </ros>
         <robot_base_frame>base_footprint${prefix}</robot_base_frame>
-        <updateRate>100</updateRate>
+        <updateRate>20</updateRate>
         <left_joint>left_wheel_joint${prefix}</left_joint>
         <right_joint>right_wheel_joint${prefix}</right_joint>
@@ -16,5 +16,5 @@
         <max_wheel_acceleration>1.0</max_wheel_acceleration>
         <publish_odom>true</publish_odom>
-        <publish_odom_tf>true</publish_odom_tf>
+        <publish_odom_tf>false</publish_odom_tf>
         <publish_wheel_tf>true</publish_wheel_tf>
         <odometry_frame>odom${prefix}</odometry_frame>

File: fru_bot_description/urdf/robots/2wd.urdf.xacro (robot description, xacro)
@@ -43,5 +43,5 @@
         prefix="${prefix}"
         side="front"
-        mass="0.01"
+        mass="0.025"
         base_length="${base_length}"
         wheel_radius="${wheel_radius}"

File: fru_bot_description/urdf/robots/FRU_bot.urdf.xacro (robot description, xacro)
@@ -10,9 +10,11 @@
         prefix="${prefix}"
         namespace="${namespace}"
-    />
+        />
     </xacro:if>
-    <xacro:robot_2wd
+    <xacro:if value="${not $(arg use_ns)}">
+        <xacro:robot_2wd
         prefix="${prefix}"
         namespace=""
-    />
+        />
+    </xacro:if>
 </robot>
