Commit message: single robot slam w/ frame_id prefix works

File: fru_bot_description/urdf/robots/FRU_bot.urdf.xacro (robot description, xacro)
@@ -3,5 +3,5 @@
     <xacro:arg name="use_ns" default="false" />
     <xacro:arg name="ns_idx" default="" />
-    <xacro:property name="prefix" value="" />
+    <xacro:property name="prefix" value="$(arg ns_idx)" />
     <xacro:property name="namespace" value="FRU_bot$(arg ns_idx)" />
     <xacro:include filename="$(find fru_bot_description)/urdf/robots/2wd.urdf.xacro"/>

File: fru_bot_description/urdf/sensors/laser.urdf.xacro (robot description, xacro)
@@ -42,5 +42,5 @@
     </joint>
     <gazebo reference="${frame_id}${prefix}">
-      <sensor type="ray" name="${frame_id}_lds_lfcd_sensor">
+      <sensor type="ray" name="${frame_id}_lds_lfcd_sensor_${prefix}">
         <always_on>true</always_on>
         <update_rate>${update_rate}</update_rate>
@@ -76,5 +76,5 @@
           <updateRate>${update_rate}</updateRate>
           <topicName>${topic_name}</topicName>
-          <frame_name>${frame_id}</frame_name>
+          <frame_name>${frame_id}${prefix}</frame_name>
           <output_type>sensor_msgs/LaserScan</output_type>
         </plugin>
