Commit message: Gazebo simulation starts, and expected topics are published at robot namespace.

File: fru_bot_description/urdf/controllers/diff_drive.urdf.xacro (robot description, xacro)
@@ -1,8 +1,9 @@
 <robot xmlns:xacro="http://ros.org/wiki/xacro">
-  <xacro:macro name="diff_drive_controller" params="prefix wheel_separation wheel_radius wheel_torque">
+  <xacro:macro name="diff_drive_controller" params="prefix namespace wheel_separation wheel_radius wheel_torque">
     <gazebo>
       <plugin name="differential_drive_controller" filename="libgazebo_ros_diff_drive.so">
         <ros>
           <argument>odom:=odom/unfiltered</argument>
+          <namespace>/${namespace}</namespace>
         </ros>
         <robot_base_frame>base_link${prefix}</robot_base_frame>
@@ -15,6 +16,6 @@
         <max_wheel_acceleration>1.0</max_wheel_acceleration>
         <publish_odom>true</publish_odom>
-        <publish_odom_tf>false</publish_odom_tf>
-        <publish_wheel_tf>true</publish_wheel_tf>
+        <publish_odom_tf>true</publish_odom_tf>
+        <publish_wheel_tf>false</publish_wheel_tf>
         <odometry_frame>odom${prefix}</odometry_frame>
         <mu1>0.5</mu1>

File: fru_bot_description/urdf/robots/2wd.urdf.xacro (robot description, xacro)
@@ -8,5 +8,5 @@
   <xacro:include filename="$(find fru_bot_description)/urdf/sensors/generic_laser.urdf.xacro" />
   <xacro:include filename="$(find fru_bot_description)/urdf/controllers/diff_drive.urdf.xacro" />
-  <xacro:macro name="robot_2wd" params="prefix">
+  <xacro:macro name="robot_2wd" params="prefix namespace">
     <xacro:base
       prefix="${prefix}"
@@ -51,10 +51,15 @@
     <xacro:imu
       prefix="${prefix}"
+      namespace="${namespace}"
     />
-    <xacro:generic_laser prefix="${prefix}">
+    <xacro:generic_laser
+      prefix="${prefix}"
+      namespace="${namespace}"
+      >
       <xacro:insert_block name="laser_pose"/>
     </xacro:generic_laser>
     <xacro:diff_drive_controller
       prefix="${prefix}"
+      namespace="${namespace}"
       wheel_separation="${wheel_pos_y * 2}"
       wheel_radius="${wheel_radius}"

File: fru_bot_description/urdf/robots/FRU_bot.urdf.xacro (robot description, xacro)
@@ -1,8 +1,11 @@
 <?xml version="1.0"?>
 <robot name="FRU_bot" xmlns:xacro="http://ros.org/wiki/xacro">
+    <xacro:property name="ns_idx" value="" />
     <xacro:property name="prefix" value="" />
+    <xacro:property name="namespace" value="FRU_bot$${ns_idx}" />
     <xacro:include filename="$(find fru_bot_description)/urdf/robots/2wd.urdf.xacro"/>
     <xacro:robot_2wd
         prefix="${prefix}"
+        namespace="${namespace}"
     />
 </robot>

File: fru_bot_description/urdf/sensors/generic_laser.urdf.xacro (robot description, xacro)
@@ -2,11 +2,12 @@
 <robot xmlns:xacro="http://ros.org/wiki/xacro">
   <xacro:include filename="$(find fru_bot_description)/urdf/sensors/laser.urdf.xacro" />
-  <xacro:macro name="generic_laser" params="prefix *origin">
+  <xacro:macro name="generic_laser" params="prefix namespace *origin">
     <xacro:laser
       prefix="${prefix}"
-      update_rate="1"
+      namespace="${namespace}"
+      update_rate="5"
       ray_count="360"
-      min_angle="-3.1416"
-      max_angle="3.1416"
+      min_angle="0.0"
+      max_angle="6.28319"
       min_range="0.12"
       max_range="3.5"
@@ -17,5 +18,5 @@
     </xacro:laser>
   </xacro:macro>
-  <xacro:macro name="generic_base_laser" params="prefix *origin">
+  <!-- <xacro:macro name="generic_base_laser" params="prefix namespace *origin">
     <xacro:laser
       prefix="${prefix}"
@@ -31,4 +32,4 @@
       <xacro:insert_block name="origin" />
     </xacro:laser>
-  </xacro:macro>
+  </xacro:macro> -->
 </robot>

File: fru_bot_description/urdf/sensors/imu.urdf.xacro (robot description, xacro)
@@ -1,4 +1,4 @@
 <robot xmlns:xacro="http://ros.org/wiki/xacro">
-  <xacro:macro name="imu" params="prefix">
+  <xacro:macro name="imu" params="prefix namespace">
     <link name="imu_link${prefix}"/>
     <joint name="imu_to_base_link${prefix}" type="fixed">
@@ -16,4 +16,5 @@
       <plugin filename="libgazebo_ros_imu_sensor.so" name="imu_plugin">
         <ros>
+          <namespace>/${namespace}</namespace>
           <remapping>~/out:=imu/data</remapping>
         </ros>

File: fru_bot_description/urdf/sensors/laser.urdf.xacro (robot description, xacro)
@@ -1,5 +1,5 @@
 <robot xmlns:xacro="http://ros.org/wiki/xacro">
   <xacro:property name="M_PI" value="3.1415926535897931" />
-  <xacro:macro name="laser" params="prefix *origin update_rate ray_count min_angle max_angle min_range max_range frame_id topic_name">
+  <xacro:macro name="laser" params="prefix namespace *origin update_rate ray_count min_angle max_angle min_range max_range frame_id topic_name">
     <link name="${frame_id}${prefix}">
       <visual>
@@ -42,5 +42,5 @@
     </joint>
     <gazebo reference="${frame_id}${prefix}">
-      <sensor type="ray" name="${frame_id}_head_hokuyo_sensor">
+      <sensor type="ray" name="${frame_id}_lds_lfcd_sensor">
         <always_on>true</always_on>
         <update_rate>${update_rate}</update_rate>
@@ -59,9 +59,15 @@
             <min>${min_range}</min>
             <max>${max_range}</max>
-            <resolution>0.01</resolution>
+            <resolution>0.015</resolution>
           </range>
+          <noise>
+          <type>gaussian</type>
+            <mean>0.0</mean>
+            <stddev>0.01</stddev>
+          </noise>
         </ray>
-        <plugin name="${frame_id}_gazebo_ros_head_hokuyo_controller" filename="libgazebo_ros_ray_sensor.so">
+        <plugin name="${frame_id}_gazebo_ros_lds_lfcd_controller" filename="libgazebo_ros_laser.so">
           <ros>
+            <namespace>/${namespace}</namespace>
             <remapping>~/out:=${topic_name}</remapping>
           </ros>

Commit message: Launches agent correctly, need to test sim.

File: fru_bot_description/urdf/controllers/diff_drive.urdf.xacro (robot description, xacro)
@@ -5,5 +5,5 @@
         <ros>
           <argument>odom:=odom/unfiltered</argument>
-          <namespace>/${namespace}</namespace>
+          <namespace>${namespace}</namespace>
         </ros>
         <robot_base_frame>base_footprint${prefix}</robot_base_frame>

File: fru_bot_description/urdf/robots/FRU_bot.urdf.xacro (robot description, xacro)
@@ -1,11 +1,18 @@
 <?xml version="1.0"?>
 <robot name="FRU_bot" xmlns:xacro="http://ros.org/wiki/xacro">
-    <xacro:property name="ns_idx" value="" />
+    <xacro:arg name="use_ns" default="false" />
+    <xacro:arg name="ns_idx" default="" />
     <xacro:property name="prefix" value="" />
-    <xacro:property name="namespace" value="FRU_bot$${ns_idx}" />
+    <xacro:property name="namespace" value="FRU_bot$(arg ns_idx)" />
     <xacro:include filename="$(find fru_bot_description)/urdf/robots/2wd.urdf.xacro"/>
-    <xacro:robot_2wd
+    <xacro:if value="$(arg use_ns)">
+        <xacro:robot_2wd
         prefix="${prefix}"
         namespace="${namespace}"
     />
+    </xacro:if>
+    <xacro:robot_2wd
+        prefix="${prefix}"
+        namespace=""
+    />
 </robot>

File: fru_bot_description/urdf/sensors/imu.urdf.xacro (robot description, xacro)
@@ -16,5 +16,5 @@
       <plugin filename="libgazebo_ros_imu_sensor.so" name="imu_plugin">
         <ros>
-          <namespace>/${namespace}</namespace>
+          <namespace>${namespace}</namespace>
           <remapping>~/out:=imu/data</remapping>
         </ros>

File: fru_bot_description/urdf/sensors/laser.urdf.xacro (robot description, xacro)
@@ -69,5 +69,5 @@
         <plugin name="${frame_id}_gazebo_ros_lds_lfcd_controller" filename="libgazebo_ros_ray_sensor.so">
           <ros>
-            <namespace>/${namespace}</namespace>
+            <namespace>${namespace}</namespace>
             <remapping>~/out:=${topic_name}</remapping>
           </ros>

Commit message: Tf remaps result in adequate simulation.

File: fru_bot_description/urdf/controllers/diff_drive.urdf.xacro (robot description, xacro)
@@ -1,4 +1,4 @@
 <robot xmlns:xacro="http://ros.org/wiki/xacro">
-  <xacro:macro name="diff_drive_controller" params="prefix namespace wheel_separation wheel_radius wheel_torque">
+  <xacro:macro name="diff_drive_controller" params="prefix namespace remap wheel_separation wheel_radius wheel_torque">
     <gazebo>
       <plugin name="differential_drive_controller" filename="libgazebo_ros_diff_drive.so">
@@ -6,4 +6,7 @@
           <argument>odom:=odom/unfiltered</argument>
           <namespace>${namespace}</namespace>
+          <xacro:if value="${remap}" >
+            <remapping>/tf:=tf</remapping>
+          </xacro:if>
         </ros>
         <robot_base_frame>base_footprint${prefix}</robot_base_frame>

File: fru_bot_description/urdf/robots/2wd.urdf.xacro (robot description, xacro)
@@ -8,5 +8,5 @@
   <xacro:include filename="$(find fru_bot_description)/urdf/sensors/generic_laser.urdf.xacro" />
   <xacro:include filename="$(find fru_bot_description)/urdf/controllers/diff_drive.urdf.xacro" />
-  <xacro:macro name="robot_2wd" params="prefix namespace">
+  <xacro:macro name="robot_2wd" params="prefix namespace remap">
     <xacro:base
       prefix="${prefix}"
@@ -62,4 +62,5 @@
       prefix="${prefix}"
       namespace="${namespace}"
+      remap="${remap}"
       wheel_separation="${wheel_pos_y * 2}"
       wheel_radius="${wheel_radius}"

File: fru_bot_description/urdf/robots/FRU_bot.urdf.xacro (robot description, xacro)
@@ -1,20 +1,13 @@
 <?xml version="1.0"?>
 <robot name="FRU_bot" xmlns:xacro="http://ros.org/wiki/xacro">
-    <xacro:arg name="use_ns" default="false" />
+    <xacro:arg name="remap" default="False" />
+    <xacro:arg name="ns" default="" />
     <xacro:arg name="ns_idx" default="" />
     <xacro:property name="prefix" value="$(arg ns_idx)" />
-    <xacro:property name="namespace" value="FRU_bot$(arg ns_idx)" />
     <xacro:include filename="$(find fru_bot_description)/urdf/robots/2wd.urdf.xacro"/>
-    <xacro:if value="$(arg use_ns)">
-        <xacro:robot_2wd
-        prefix="${prefix}"
-        namespace="${namespace}"
-        />
-    </xacro:if>
-    <xacro:if value="${not $(arg use_ns)}">
-        <xacro:robot_2wd
-        prefix="${prefix}"
-        namespace=""
-        />
-    </xacro:if>
+    <xacro:robot_2wd
+    prefix="${prefix}"
+    namespace="$(arg ns)"
+    remap="$(arg remap)"
+    />
 </robot>
